File: Hardware/Production/MicroMod-Teensy-Panel.brd (EAGLE design)
At the start: 195 x 82.5 mm, 1302 parts, among them J1 MICROMOD-2222, J10 MICROMOD-2222, J11 MICROMOD-2222, J12 MICROMOD-2222, J13 MICROMOD-2222, J14 MICROMOD-2222, J15 MICROMOD-2222, J16 MICROMOD-2222, J2 MICROMOD-2222, J3 MICROMOD-2222, J4 MICROMOD-2222, J5 MICROMOD-2222, J6 MICROMOD-2222, J7 MICROMOD-2222, J8 MICROMOD-2222, J9 MICROMOD-2222, Q1 20V/4.2A/52mΩ/1.4W, Q10 20V/0.2A/8MHz/1.2Ω/1Vth, Q11 20V/4.2A/52mΩ/1.4W, Q12 20V/0.2A/8MHz/1.2Ω/1Vth, Q13 20V/4.2A/52mΩ/1.4W, Q14 20V/0.2A/8MHz/1.2Ω/1Vth, Q15 20V/4.2A/52mΩ/1.4W, Q16 20V/0.2A/8MHz/1.2Ω/1Vth, Q17 20V/4.2A/52mΩ/1.4W, Q18 20V/0.2A/8MHz/1.2Ω/1Vth, Q19 20V/4.2A/52mΩ/1.4W, Q2 20V/0.2A/8MHz/1.2Ω/1Vth, Q20 20V/0.2A/8MHz/1.2Ω/1Vth, Q21 20V/4.2A/52mΩ/1.4W, Q22 20V/0.2A/8MHz/1.2Ω/1Vth, Q23 20V/4.2A/52mΩ/1.4W, Q24 20V/0.2A/8MHz/1.2Ω/1Vth, Q25 20V/4.2A/52mΩ/1.4W, Q26 20V/0.2A/8MHz/1.2Ω/1Vth, Q27 20V/4.2A/52mΩ/1.4W, Q28 20V/0.2A/8MHz/1.2Ω/1Vth, Q29 20V/4.2A/52mΩ/1.4W, Q3 20V/4.2A/52mΩ/1.4W, Q30 20V/0.2A/8MHz/1.2Ω/1Vth, Q31 20V/4.2A/52mΩ/1.4W, Q32 20V/0.2A/8MHz/1.2Ω/1Vth, Q4 20V/0.2A/8MHz/1.2Ω/1Vth, Q5 20V/4.2A/52mΩ/1.4W, Q6 20V/0.2A/8MHz/1.2Ω/1Vth, Q7 20V/4.2A/52mΩ/1.4W, Q8 20V/0.2A/8MHz/1.2Ω/1Vth, Q9 20V/4.2A/52mΩ/1.4W, U1 IMXRT1062DV10X10, U10 IMXRT1062DV10X10, U11 MKL02Z32VFG4, U12 W25QXX128MBIT-6X5, U13 IMXRT1062DV10X10, U14 MKL02Z32VFG4, U15 W25QXX128MBIT-6X5, U16 IMXRT1062DV10X10, U17 MKL02Z32VFG4, U18 W25QXX128MBIT-6X5, U19 IMXRT1062DV10X10, U2 IMXRT1062DV10X10, U20 MKL02Z32VFG4, U21 W25QXX128MBIT-6X5, U22 IMXRT1062DV10X10, U23 MKL02Z32VFG4, U24 W25QXX128MBIT-6X5, U25 IMXRT1062DV10X10, U26 MKL02Z32VFG4, U27 W25QXX128MBIT-6X5, U28 IMXRT1062DV10X10, U29 MKL02Z32VFG4, U3 MKL02Z32VFG4, U30 W25QXX128MBIT-6X5, U31 IMXRT1062DV10X10, U32 MKL02Z32VFG4, U33 W25QXX128MBIT-6X5, U34 IMXRT1062DV10X10, U35 MKL02Z32VFG4, U36 W25QXX128MBIT-6X5, U37 IMXRT1062DV10X10, U38 MKL02Z32VFG4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

Commit message: Add panel files for v15 with ENIG finish notes
Parts:
- removed FRAME1, FRAME10, FRAME11, FRAME12, FRAME13, FRAME14, FRAME15, FRAME16, FRAME2, FRAME3, FRAME4, FRAME5, FRAME6, FRAME7, FRAME8, FRAME9: FRAME-LEDGER, SparkFun-Aesthetics:CREATIVE_COMMONS
- removed LOGO17, LOGO19, LOGO21, LOGO23, LOGO25, LOGO27, LOGO29, LOGO31: SFE_LOGO_NAME_FLAME.1_INCH, SparkFun-Aesthetics:SFE_LOGO_NAME_FLAME_.1
- removed LOGO18, LOGO20, LOGO22, LOGO24, LOGO26, LOGO28, LOGO30, LOGO32: OSHW-LOGONO_SILK, SparkFun-Aesthetics:DUMMY
- LOGO10, LOGO12, LOGO14, LOGO16, LOGO2, LOGO4, LOGO6, LOGO8: value OSHW-LOGONO_SILK -> SFE_LOGO_NAME_FLAME.1_INCH; device SparkFun-Aesthetics:DUMMY -> SparkFun-Aesthetics:SFE_LOGO_NAME_FLAME_.1
- moved LOGO10 96.6 mm to (37.3, 51.7), flipped to the bottom, turned to 180 degrees
- moved LOGO8 91.5 mm to (160.7, 18.1), flipped to the bottom
- moved LOGO9 86.2 mm to (15.3, 51.7), turned to 180 degrees
- moved LOGO12 84.0 mm to (81.3, 51.7), flipped to the bottom, turned to 180 degrees
- moved LOGO14 75.7 mm to (125.3, 51.7), flipped to the bottom, turned to 180 degrees
- moved LOGO16 73.4 mm to (169.3, 51.7), flipped to the bottom, turned to 180 degrees
- moved LOGO6 72.3 mm to (116.7, 18.1), flipped to the bottom
- moved LOGO11 66.5 mm to (59.3, 51.7), turned to 180 degrees
- moved LOGO7 66.0 mm to (138.7, 18.1)
- moved LOGO4 55.3 mm to (72.7, 18.1), flipped to the bottom
- moved LOGO13 48.8 mm to (103.3, 51.7), turned to 180 degrees
- moved LOGO5 44.0 mm to (94.7, 18.1)
- moved LOGO2 43.0 mm to (28.7, 18.1), flipped to the bottom
- moved LOGO15 36.2 mm to (147.3, 51.7), turned to 180 degrees
- moved LOGO3 22.0 mm to (50.7, 18.1)
Connections:
- net MISO/1 renamed CIPO/1
- net MISO/10 renamed CIPO/10
- net MISO/11 renamed CIPO/11
- net MISO/12 renamed CIPO/12
- net MISO/13 renamed CIPO/13
- net MISO/14 renamed CIPO/14
- net MISO/15 renamed CIPO/15
- net MISO/16 renamed CIPO/16
- net MISO/2 renamed CIPO/2
- net MISO/3 renamed CIPO/3
- net MISO/4 renamed CIPO/4
- net MISO/5 renamed CIPO/5
- net MISO/6 renamed CIPO/6
- net MISO/7 renamed CIPO/7
- net MISO/8 renamed CIPO/8
- net MISO/9 renamed CIPO/9
- net MOSI/1 renamed COPI/1
- net MOSI/10 renamed COPI/10
- net MOSI/11 renamed COPI/11
- net MOSI/12 renamed COPI/12
- net MOSI/13 renamed COPI/13
- net MOSI/14 renamed COPI/14
- net MOSI/15 renamed COPI/15
- net MOSI/16 renamed COPI/16
- net MOSI/2 renamed COPI/2
- net MOSI/3 renamed COPI/3
- net MOSI/4 renamed COPI/4
- net MOSI/5 renamed COPI/5
- net MOSI/6 renamed COPI/6
- net MOSI/7 renamed COPI/7
- net MOSI/8 renamed COPI/8
- net MOSI/9 renamed COPI/9
