File: Hardware/MicroMod-Teensy.sch (EAGLE design)
At the start: 71 parts, among them J1 MICROMOD-2222, Q1 20V/4.2A/52mΩ/1.4W, Q2 20V/0.2A/8MHz/1.2Ω/1Vth, U1 IMXRT1062DV10X10, U3 MKL02Z32VFG4, U4 W25QXX128MBIT-6X5, Y1 32.768kHz, Y2 24MHz

Commit message: Switch layers 2/15 to put ground under xtals. Increase GND plane on layer 15.
Connections:
- net N$31 renamed 32KHZ_2
- net N$32 renamed 32KHZ_1
- net N$4 renamed 24MHZ_1
- net N$5 renamed 24MHZ_2
Changed lines of the file:
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@@
 <?xml version="1.0" encoding="utf-8"?>
 <!DOCTYPE eagle SYSTEM "eagle.dtd">
-<eagle version="9.6.0">
+<eagle version="9.6.2">
 <drawing>
 <settings>
@@
 </segment>
 </net>
-<net name="N$31" class="0">
+<net name="32KHZ_2" class="0">
 <segment>
 <pinref part="U1" gate="U1" pin="RTC_XTALO"/>
@@
 </segment>
 </net>
-<net name="N$32" class="0">
+<net name="32KHZ_1" class="0">
 <segment>
 <pinref part="U1" gate="U1" pin="RTC_XTALI"/>
@@
 </segment>
 </net>
-<net name="N$4" class="0">
+<net name="24MHZ_1" class="0">
 <segment>
 <pinref part="U1" gate="U1" pin="XTALO"/>
@@
 </segment>
 </net>
-<net name="N$5" class="0">
+<net name="24MHZ_2" class="0">
 <segment>
 <pinref part="U1" gate="U1" pin="XTALI"/>

Commit message: Increase TP size and relocate to more open areas
Parts:
- TP1, TP10, TP11, TP2, TP3, TP4, TP5, TP6, TP7, TP8, TP9: value TEST-POINT2 -> TEST-POINT3; device SparkFun-Connectors:TEST-POINT2 -> SparkFun-Connectors:TEST-POINT3

Commit message: Connect 3.3V_Controlled to peripherals. Increase internal power trace widths.
Parts:
- added TP12, TP13: TEST-POINT3, SparkFun-Connectors:TEST-POINT3
Connections:
- net N$3 renamed DCDC_IN
- net N$9 renamed DCDC_LP
- net 3.3V: now also TP13.1; no longer C28.1, C29.1, D5.A, FB2.1, U3.VDD, U4.VDD
- net 3.3V_CONTROLLED: now also C28.1, C29.1, D5.A, FB2.1, TP12.1, U3.VDD, U4.VDD
Other:
- moved on the sheet: C28, D5, R5, R7, TP1, TP10, TP11, TP2, TP3, TP4, TP5, TP6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
